File: TOSV-SENSOR-REF V1.0/CAD/TMCM-0021 v1.0.kicad_pcb (KiCad board)
At the start: 4 copper layers, 34 x 56 mm, 67 parts, among them IC101 ADS7142IRUGR, IC102 SN65HVD1781D, J101 Conn_01x10, J102 Conn_01x10, J103 Conn_01x02, U101 SSCDRRN160MGAA5, U102 SM9333-BCE-S-125-000, U103 SSCDRRN160MGAA5, U201 MAX9095AUD+T

Commit message: Silkscree Update
Parts:
- removed the G*** at (3.72, -32.9)
- added G***: LOGO, KiCad library:New trinamic logo (maxim), F.Cu at (5.08, -33.0)
Other:
- board text added: "(TMCM-0021 v1.0)"
- board text added: "TOSV-SENSOR-REF"
- board text removed: "TMCM-0021 v1.0"
